File: ClaudeMicro.kicad_pcb (KiCad board)
At the start: 4 copper layers, 90 x 90 mm, 97 parts, among them J1 USB-C_SMD-TYPE-C-31-M-12_1, J2 SWD, SW1 CONN-SMD_HOTPLUGPAKAGE__C9900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, SW10 CONN-SMD_HOTPLUGPAKAGE__C9900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, SW11 CONN-SMD_HOTPLUGPAKAGE__C9900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, SW12 CONN-SMD_HOTPLUGPAKAGE__C9900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, SW13 SW-SMD_4P-L5.1-W5.1-P3.70-LS6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, SW14 CONN-SMD_HOTPLUGPAKAGE__C9900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, SW2 CONN-SMD_HOTPLUGPAKAGE__C9900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, SW3 CONN-SMD_HOTPLUGPAKAGE__C9900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, SW4 CONN-SMD_HOTPLUGPAKAGE__C9900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, SW5 CONN-SMD_HOTPLUGPAKAGE__C9900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, SW6 CONN-SMD_HOTPLUGPAKAGE__C9900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, SW7 CONN-SMD_HOTPLUGPAKAGE__C9900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, SW8 CONN-SMD_HOTPLUGPAKAGE__C9900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, SW9 CONN-SMD_HOTPLUGPAKAGE__C9900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, U1 LQFN-56_L7.0-W7.0-P0.4-EP, U2 SOIC-8_L5.3-W5.3-P1.27-LS8.0-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, U3 SOT-223-3_L6.5-W3.4-P2.30-LS7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, U4 SOT-23-5_L3.0-W1.7-P0.95-LS2.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, U6 SOT-23-6_L2.9-W1.6-P0.95-LS2.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, Y1 CRYSTAL-SMD_4P-L3.2-W2.5-BL

Commit message: Remove dead scripts
Parts:
- added D16: LED-SMD_4P-L3.2-W2.8-LS5.9_SK6812MINI-E, LED-SMD_4P-L3.2-W2.8-LS5.9_SK6812MINI-E, B.Cu at (13.5, 81.5)
Connections:
- D15 pad 4: unconnected-(D15-DOUT-Pad4) -> LED_D13
Routing:
- net LED_D13: track 0.00 -> 86.1 mm, vias 0 -> 2
- net K6: track 78.4 -> 57.0 mm
- net K10: track 58.1 -> 42.2 mm, vias 3 -> 0
- net XIN: track 24.0 -> 38.2 mm
- net SWDIO: track 35.5 -> 27.4 mm
- net GND: track 128.9 -> 136.8 mm, vias 183 -> 182
- net ENC_SW: track 87.9 -> 95.6 mm
- net JOY_A: track 89.4 -> 95.9 mm, vias 2 -> 1
- net LED_DATA: track 102.8 -> 96.5 mm
- net K7: track 48.4 -> 54.1 mm
- net QSPI_SS: track 45.9 -> 40.2 mm
- net RUN: track 34.0 -> 38.6 mm
- net K9: track 37.6 -> 33.1 mm
- net ENC_A: track 81.7 -> 77.6 mm
- net AUX1: track 60.8 -> 64.8 mm, vias 3 -> 2
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
Commit message: Move LEDs under keys
Parts:
- moved D3 15.1 mm to (16.0, 29.9)
- moved D4 15.1 mm to (35.3, 29.9)
- moved D5 15.1 mm to (54.7, 29.9)
- moved D6 15.1 mm to (74.0, 29.9)
- moved D10 15.1 mm to (16.0, 48.5)
- moved D11 15.1 mm to (35.3, 48.5)
- moved D12 15.1 mm to (54.7, 48.5)
- moved D13 15.1 mm to (74.0, 48.5)
- moved D1 15.1 mm to (35.3, 11.2)
- moved D2 15.1 mm to (54.7, 11.2)
- moved D16 14.5 mm to (16.0, 67.2)
- moved D15 10.2 mm to (74.0, 67.2)
- moved D14 3.77 mm to (45.0, 67.2)
Routing:
- net VBUS: track 244.8 -> 278.2 mm, vias 25 -> 27
- net GND: track 136.8 -> 156.0 mm, vias 182 -> 167
- net LED_D13: track 86.1 -> 67.4 mm
- net LED_D1: track 22.8 -> 7.94 mm
- net K6: track 57.0 -> 71.8 mm, vias 2 -> 3
- net LED_D12: track 38.9 -> 24.7 mm, vias 2 -> 0
- net XIN: track 38.2 -> 26.4 mm
- net XOUT_XTAL: track 6.96 -> 17.4 mm
- net CC2: track 20.4 -> 29.0 mm
- net K7: track 54.1 -> 46.8 mm
- net JOY_D: track 81.7 -> 88.5 mm, vias 1 -> 2
- net K12: track 31.7 -> 38.3 mm
- net LED_DATA: track 96.5 -> 89.9 mm
- net LED_D11: track 39.2 -> 45.3 mm
- net RUN: track 38.6 -> 32.5 mm
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
Commit message: Add changelog, silk license
Other:
- board text added: "ClaudeMicro v0.1 · OSHW · CERN-OHL-S v2 · github.com/Brillar0101"
- board text removed: "ClaudeMicro v0.1 · OSHW · github.com/Brillar0101"
Changed lines of the file:
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@@
 		)
 	)
-	(gr_text "ClaudeMicro v0.1 · OSHW · github.com/Brillar0101"
+	(gr_text "ClaudeMicro v0.1 · OSHW · CERN-OHL-S v2 · github.com/Brillar0101"
 		(at 86.5 45 90)
 		(layer "B.SilkS")
