File: hardware/ClaudeMicro.kicad_sch (KiCad schematic)
At the start: 82 parts, among them J1 USB-C, J2 SWD, SW1 K1, SW10 K10, SW11 K11, SW12 K12, SW13 BOOTSEL, SW2 K2, SW3 K3, SW4 K4, SW5 K5, SW6 K6, SW7 K7, SW8 K8, SW9 K9, U1 RP2040, U2 W25Q128JVSIQ, U3 AMS1117-3.3, U4 74AHCT1G125, U5 TTP223-BA6, U6 USBLC6-2SC6, Y1 ABM8-272-T3

Commit message: fix: clear DRC errors, adjust silkscreen, regenerate fab package
- Add GND stitching via at (55.605, 88.624) connecting orphan B.Cu
  island carrying C12 pad 2 (decoupling cap ground was floating)
- Remove 9 redundant vias drilled on top of ENC1/JS1/J1 PTH pad holes
- Convert 26 zero-annular-ring switch alignment posts (SW1-SW14) to NPTH
- Silkscreen text repositioned; clears silk_edge_clearance warning
- Schematic resaved by KiCad 10 (format normalization, sch_revision V0.1)
- Regenerate gerbers, drills, CPL from DRC-clean board (0 errors)
Other:
- moved on the sheet: C10, C11, C12, C13, C14, C16, C17, C3, C4, C5, C6, C7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
