File: hardware/AgentDeck.kicad_sch (KiCad schematic)
At the start: 82 parts, among them J1 USB-C, J2 SWD, SW1 K1, SW10 K10, SW11 K11, SW12 K12, SW13 BOOTSEL, SW2 K2, SW3 K3, SW4 K4, SW5 K5, SW6 K6, SW7 K7, SW8 K8, SW9 K9, U1 RP2040, U2 W25Q128JVSIQ, U3 AMS1117-3.3, U4 74AHCT1G125, U5 TTP223-BA6, U6 USBLC6-2SC6, Y1 ABM8-272-T3

Commit message: rename to agentdeck 1.0.0
The product is renamed from ClaudeMicro to AgentDeck for 1.0.0. "Claude" is
Anthropic's trademark and this ships as OSHWA-marked open hardware with the
name on the silk; "Micro" also stopped describing a 150x110 mm V4 deck. Note
AgentDeck collides with an existing project (github.com/puritysb/AgentDeck) -
chosen anyway.

Renamed across board, schematic, netlist, libraries, firmware, host bridge and
docs. Silk reads AGENTDECK and AgentDeck v1.0.0. Generated gerbers under
fab/gerbers are left alone: they are the artifact of the released v0.1.0 and
should be regenerated rather than string-edited.

Also in this commit, all verified 0 errors / 0 unconnected:

- silkscreen pass (tools/silk_pass.py, silk_finish.py, fix_silk_font.py):
  silk_over_copper 79 -> 0, silk_overlap 7 -> 0, text_height 4 -> 0. Silk is
  Red Hat Mono bold; bold and 1.3 mm on the three longest strings are not
  cosmetic - KiCad flags Red Hat Mono Regular at 1.0 mm as insufficient stroke
  weight, the outline-font tradeoff a stroke font avoids. Re-running the pass
  is a no-op, so it is safe after any placement change.

- placement pass (tools/placement_pass.py): three fiducials placed
  asymmetrically >=5 mm from the edges, and C10 moved +0.75/-2.25 mm. C9 and
  C10 were not merely close, their bodies overlapped - two 0603 caps in the
  same space, invisible to DRC because both are +3V3/GND so no clearance rule
  applies. Only C10 moved; the outline and every part the case mates with are
  untouched.

- fab/AgentDeck-BOM-v1.0.0.csv. Records that C22967 is 27k, not the 27R the
  old BOM claimed for the USB series resistors - at 27k USB would not
  enumerate. Correct part is C25190. Also records what LCSC cannot supply:
  the Kailh hot-swap socket (C5333465 discontinued) and the SKQUCAA010
  joystick, plus switches and keycaps which were never LCSC lines.

- docs/img: top and bottom board renders.
Parts:
- J2: footprint ClaudeMicro:ProgPads_1x4 -> AgentDeck:ProgPads_1x4; symbol ClaudeMicro_Custom:ProgPads_1x4 -> AgentDeck_Custom:ProgPads_1x4
- JS1: footprint ClaudeMicro:SKQUCAA010 -> AgentDeck:SKQUCAA010; symbol ClaudeMicro_Custom:SKQUCAA010 -> AgentDeck_Custom:SKQUCAA010
- TP1: footprint ClaudeMicro:TouchPad_D12 -> AgentDeck:TouchPad_D12; symbol ClaudeMicro_Custom:TouchPad -> AgentDeck_Custom:TouchPad
Other:
- title: Claude Micro -> AgentDeck
