File: v4/hardware/ClaudeMicroV4.kicad_sch (KiCad schematic)
At the start: 142 parts, among them J1 TYPE-C-31-M-12, J2 JST-PH-2 LiPo, J3 ProgPads 3V3/TX/GND/RX, J4 JST-PH-2 Speaker, Q1 AO3401A, SW1 ChocV1, SW10 ChocV1, SW11 ChocV1, SW12 ChocV1, SW13 ChocV1, SW14 ChocV1, SW15 ChocV1, SW16 ChocV1, SW17 ChocV1, SW18 ChocV1, SW19 ChocV1, SW2 ChocV1, SW20 ChocV1, SW21 ChocV1, SW22 ChocV1, SW23 ChocV1, SW24 ChocV1, SW25 MSK12C02, SW26 SW_PUSH, SW27 SW_PUSH, SW3 ChocV1, SW4 ChocV1, SW5 ChocV1, SW6 ChocV1, SW7 ChocV1, SW8 ChocV1, SW9 ChocV1, U1 ESP32-S3-WROOM-1-N8R2, U2 SN74AHCT1G125, U3 USBLC6-2SC6, U4 TP4056, U5 ME6211C33, U6 NS4168

Commit message: route v4 board
Phase 2 complete: the V4 board is fully routed and DRC-clean (0 errors,
0 unconnected, 970 tracks, 380 vias).

freerouting closed 167/172 connections and stalled at pass 8; finish_v4
imported the SES, poured GND and VSYS_SW, and bridged 30 pour clusters.
knit_maze's A* recovered VSYS_SW C6.1. Three defects were left over and
are fixed here:

- USB_DP short. phase 4b0's add_seg() wrote tracks with no clearance
  guard - the only unguarded path in that block - driving the B6 descent
  straight through the VBAT_SNS run. add_seg now builds the model lazily
  (so it sees the del_box rip-ups above it) and checks seg_clear before
  committing, like the BESPOKE block. Without this the pipeline recreates
  the short on every run.

- C3 floating. Its ground pad reached only an isolated pour island: F.Cu
  fenced by the +3V3 rail (deleting it splits the rail, moving it does
  not help since any C4->C3 path crosses the same corridor) and B.Cu
  shredded into non-main slivers by seven bus lanes, with zero island
  points over main B fill - so no via or jumper existed. C3 is a bulk cap
  20 mm from U1's supply pin, so it moved to dy=2.6/dx=-0.8 with a feed
  tapped off the C4 run. knit_final then bridged GND C5.2, which had
  failed every earlier attempt.

- 14 stitching vias drilled dead centre on same-net PTH pads (J1, U4, U6,
  both encoders). A PTH pad already joins both layers, so these were
  duplicate drill hits.

The 37 VSYS_SW via_dangling warnings are left alone deliberately: those
vias stitch the pour between layers, and removing them splits the rail
into 6 clusters.
Parts:
- U6: footprint V3:ESOP-8_TP4056 -> V4:ESOP-8_NS4168
Changed lines of the file:
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@@
 			)
 		)
-		(property "Footprint" "V3:ESOP-8_TP4056"
+		(property "Footprint" "V4:ESOP-8_NS4168"
 			(at 900.0 70.0 0)
 			(effects
