File: v4/hardware/AgentDeckV4.kicad_pcb (KiCad board)
At the start: 2 copper layers, 150 x 110 mm, 148 parts, among them J1 USB-C_SMD-TYPE-C-31-M-12_1, J2 JST_PH_S2B-PH-SM4-TB_1x02-1MP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, J3 SWD, J4 JST_PH_S2B-PH-SM4-TB_1x02-1MP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, Q1 SOT-23, SW1 ChocV1_Direct, SW10 ChocV1_Direct, SW11 ChocV1_Direct, SW12 ChocV1_Direct, SW13 ChocV1_Direct, SW14 ChocV1_Direct, SW15 ChocV1_Direct, SW16 ChocV1_Direct, SW17 ChocV1_Direct, SW18 ChocV1_Direct, SW19 ChocV1_Direct, SW2 ChocV1_Direct, SW20 ChocV1_Direct, SW21 ChocV1_Direct, SW22 ChocV1_Direct, SW23 ChocV1_Direct, SW24 ChocV1_Direct, SW25 MSK12C02, SW26 SW-SMD_4P-L5.1-W5.1-P3.70-LS6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, SW27 SW-SMD_4P-L5.1-W5.1-P3.70-LS6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, SW3 ChocV1_Direct, SW4 ChocV1_Direct, SW5 ChocV1_Direct, SW6 ChocV1_Direct, SW7 ChocV1_Direct, SW8 ChocV1_Direct, SW9 ChocV1_Direct, U1 WIRELM-SMD_ESP32-S3-WROOM-1, U2 SOT-23-5_L3.0-W1.7-P0.95-LS2.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, U3 SOT-23-6_L2.9-W1.6-P0.95-LS2.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, U4 ESOP-8_TP4056, U5 SOT-23-5_L3.0-W1.7-P0.95-LS2.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, U6 ESOP-8_NS4168

Commit message: rename to agentdeck 1.0.0
The product is renamed from ClaudeMicro to AgentDeck for 1.0.0. "Claude" is
Anthropic's trademark and this ships as OSHWA-marked open hardware with the
name on the silk; "Micro" also stopped describing a 150x110 mm V4 deck. Note
AgentDeck collides with an existing project (github.com/puritysb/AgentDeck) -
chosen anyway.

Renamed across board, schematic, netlist, libraries, firmware, host bridge and
docs. Silk reads AGENTDECK and AgentDeck v1.0.0. Generated gerbers under
fab/gerbers are left alone: they are the artifact of the released v0.1.0 and
should be regenerated rather than string-edited.

Also in this commit, all verified 0 errors / 0 unconnected:

- silkscreen pass (tools/silk_pass.py, silk_finish.py, fix_silk_font.py):
  silk_over_copper 79 -> 0, silk_overlap 7 -> 0, text_height 4 -> 0. Silk is
  Red Hat Mono bold; bold and 1.3 mm on the three longest strings are not
  cosmetic - KiCad flags Red Hat Mono Regular at 1.0 mm as insufficient stroke
  weight, the outline-font tradeoff a stroke font avoids. Re-running the pass
  is a no-op, so it is safe after any placement change.

- placement pass (tools/placement_pass.py): three fiducials placed
  asymmetrically >=5 mm from the edges, and C10 moved +0.75/-2.25 mm. C9 and
  C10 were not merely close, their bodies overlapped - two 0603 caps in the
  same space, invisible to DRC because both are +3V3/GND so no clearance rule
  applies. Only C10 moved; the outline and every part the case mates with are
  untouched.

- fab/AgentDeck-BOM-v1.0.0.csv. Records that C22967 is 27k, not the 27R the
  old BOM claimed for the USB series resistors - at 27k USB would not
  enumerate. Correct part is C25190. Also records what LCSC cannot supply:
  the Kailh hot-swap socket (C5333465 discontinued) and the SKQUCAA010
  joystick, plus switches and keycaps which were never LCSC lines.

- docs/img: top and bottom board renders.
Other:
- board text added: "AgentDeck V4 - princetekki.com"
- board text added: "AgentDeckV4 ESP32-S3-WROOM-1"
- board text removed: "ClaudeMicro V4 - princetekki.com"
- board text removed: "ClaudeMicroV4 ESP32-S3-WROOM-1"
Changed lines of the file:
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@@
 		)
 		(embedded_fonts no)
-		(model "/Users/barakaeli/kicad-projects/claude-micro/hardware/JLC.3dshapes/SW-SMD_4P-L5.1-W5.1-P3.70-LS6.5-TL_H1.5.wrl"
+		(model "/Users/barakaeli/kicad-projects/agentdeck/hardware/JLC.3dshapes/SW-SMD_4P-L5.1-W5.1-P3.70-LS6.5-TL_H1.5.wrl"
 			(offset
 				(xyz 0 0 0)
@@
 		)
 		(embedded_fonts no)
-		(model "/Users/barakaeli/kicad-projects/claude-micro/hardware/JLC.3dshapes/SOT-23-6_L2.9-W1.6-H1.5-LS2.8-P0.95.wrl"
+		(model "/Users/barakaeli/kicad-projects/agentdeck/hardware/JLC.3dshapes/SOT-23-6_L2.9-W1.6-H1.5-LS2.8-P0.95.wrl"
 			(offset
 				(xyz 0 0 0)
@@
 		)
 		(embedded_fonts no)
-		(model "/Users/barakaeli/kicad-projects/claude-micro/hardware/JLC.3dshapes/SW-SMD_4P-L5.1-W5.1-P3.70-LS6.5-TL_H1.5.wrl"
+		(model "/Users/barakaeli/kicad-projects/agentdeck/hardware/JLC.3dshapes/SW-SMD_4P-L5.1-W5.1-P3.70-LS6.5-TL_H1.5.wrl"
 			(offset
 				(xyz 0 0 0)
@@
 		)
 		(embedded_fonts no)
-		(model "/Users/barakaeli/kicad-projects/claude-micro/hardware/JLC.3dshapes/SW-TH_EC11E1820402-L11.7-W12.0-H24.5-P2.5-LS14.5.wrl"
+		(model "/Users/barakaeli/kicad-projects/agentdeck/hardware/JLC.3dshapes/SW-TH_EC11E1820402-L11.7-W12.0-H24.5-P2.5-LS14.5.wrl"
 			(offset
 				(xyz 0 0 0)
@@
 		)
 		(embedded_fonts no)
-		(model "/Users/barakaeli/kicad-projects/claude-micro/hardware/JLC.3dshapes/USB-C_SMD-TYPE-C-31-M-12_1.wrl"
+		(model "/Users/barakaeli/kicad-projects/agentdeck/hardware/JLC.3dshapes/USB-C_SMD-TYPE-C-31-M-12_1.wrl"
 			(offset
 				(xyz 0 0 0)
@@
 		)
 		(embedded_fonts no)
-		(model "/Users/barakaeli/kicad-projects/claude-micro/hardware/JLC.3dshapes/SOT-23-5_L2.9-W1.6-H1.1-LS2.8-P0.95.wrl"
+		(model "/Users/barakaeli/kicad-projects/agentdeck/hardware/JLC.3dshapes/SOT-23-5_L2.9-W1.6-H1.1-LS2.8-P0.95.wrl"
 			(offset
 				(xyz 0 0 0)
@@
 		)
 		(embedded_fonts no)
-		(model "/Users/barakaeli/kicad-projects/claude-micro/hardware/JLC.3dshapes/SW-TH_EC11E1820402-L11.7-W12.0-H24.5-P2.5-LS14.5.wrl"
+		(model "/Users/barakaeli/kicad-projects/agentdeck/hardware/JLC.3dshapes/SW-TH_EC11E1820402-L11.7-W12.0-H24.5-P2.5-LS14.5.wrl"
 			(offset
 				(xyz 0 0 0)
@@
 		)
 		(embedded_fonts no)
-		(model "/Users/barakaeli/kicad-projects/claude-micro/hardware/JLC.3dshapes/LED-SMD_4P-L3.2-W2.8-LS5.9_SK6812MINI-E.wrl"
+		(model "/Users/barakaeli/kicad-projects/agentdeck/hardware/JLC.3dshapes/LED-SMD_4P-L3.2-W2.8-LS5.9_SK6812MINI-E.wrl"
 			(offset
 				(xyz 0 0 0)
@@
 		)
 		(embedded_fonts no)
-		(model "/Users/barakaeli/kicad-projects/claude-micro/hardware/JLC.3dshapes/LED-SMD_4P-L3.2-W2.8-LS5.9_SK6812MINI-E.wrl"
+		(model "/Users/barakaeli/kicad-projects/agentdeck/hardware/JLC.3dshapes/LED-SMD_4P-L3.2-W2.8-LS5.9_SK6812MINI-E.wrl"
 			(offset
 				(xyz 0 0 0)
@@
 		)
 		(embedded_fonts no)
-		(model "/Users/barakaeli/kicad-projects/claude-micro/hardware/JLC.3dshapes/LED-SMD_4P-L3.2-W2.8-LS5.9_SK6812MINI-E.wrl"
+		(model "/Users/barakaeli/kicad-projects/agentdeck/hardware/JLC.3dshapes/LED-SMD_4P-L3.2-W2.8-LS5.9_SK6812MINI-E.wrl"
 			(offset
 				(xyz 0 0 0)
@@
 		)
 		(embedded_fonts no)
-		(model "/Users/barakaeli/kicad-projects/claude-micro/hardware/JLC.3dshapes/LED-SMD_4P-L3.2-W2.8-LS5.9_SK6812MINI-E.wrl"
+		(model "/Users/barakaeli/kicad-projects/agentdeck/hardware/JLC.3dshapes/LED-SMD_4P-L3.2-W2.8-LS5.9_SK6812MINI-E.wrl"
 			(offset
 				(xyz 0 0 0)
@@
 		)
 		(embedded_fonts no)
-		(model "/Users/barakaeli/kicad-projects/claude-micro/hardware/JLC.3dshapes/LED-SMD_4P-L3.2-W2.8-LS5.9_SK6812MINI-E.wrl"
+		(model "/Users/barakaeli/kicad-projects/agentdeck/hardware/JLC.3dshapes/LED-SMD_4P-L3.2-W2.8-LS5.9_SK6812MINI-E.wrl"
 			(offset
 				(xyz 0 0 0)
@@
 		)
 		(embedded_fonts no)
-		(model "/Users/barakaeli/kicad-projects/claude-micro/hardware/JLC.3dshapes/LED-SMD_4P-L3.2-W2.8-LS5.9_SK6812MINI-E.wrl"
+		(model "/Users/barakaeli/kicad-projects/agentdeck/hardware/JLC.3dshapes/LED-SMD_4P-L3.2-W2.8-LS5.9_SK6812MINI-E.wrl"
 			(offset
 				(xyz 0 0 0)
@@
 		)
 		(embedded_fonts no)
-		(model "/Users/barakaeli/kicad-projects/claude-micro/hardware/JLC.3dshapes/LED-SMD_4P-L3.2-W2.8-LS5.9_SK6812MINI-E.wrl"
+		(model "/Users/barakaeli/kicad-projects/agentdeck/hardware/JLC.3dshapes/LED-SMD_4P-L3.2-W2.8-LS5.9_SK6812MINI-E.wrl"
 			(offset
 				(xyz 0 0 0)
@@
 		)
 		(embedded_fonts no)
-		(model "/Users/barakaeli/kicad-projects/claude-micro/hardware/JLC.3dshapes/LED-SMD_4P-L3.2-W2.8-LS5.9_SK6812MINI-E.wrl"
+		(model "/Users/barakaeli/kicad-projects/agentdeck/hardware/JLC.3dshapes/LED-SMD_4P-L3.2-W2.8-LS5.9_SK6812MINI-E.wrl"
 			(offset
 				(xyz 0 0 0)
@@
 		)
 		(embedded_fonts no)
-		(model "/Users/barakaeli/kicad-projects/claude-micro/hardware/JLC.3dshapes/LED-SMD_4P-L3.2-W2.8-LS5.9_SK6812MINI-E.wrl"
+		(model "/Users/barakaeli/kicad-projects/agentdeck/hardware/JLC.3dshapes/LED-SMD_4P-L3.2-W2.8-LS5.9_SK6812MINI-E.wrl"
 			(offset
 				(xyz 0 0 0)
@@
 		)
 		(embedded_fonts no)
-		(model "/Users/barakaeli/kicad-projects/claude-micro/hardware/JLC.3dshapes/LED-SMD_4P-L3.2-W2.8-LS5.9_SK6812MINI-E.wrl"
+		(model "/Users/barakaeli/kicad-projects/agentdeck/hardware/JLC.3dshapes/LED-SMD_4P-L3.2-W2.8-LS5.9_SK6812MINI-E.wrl"
 			(offset
 				(xyz 0 0 0)
@@
 		)
 		(embedded_fonts no)
-		(model "/Users/barakaeli/kicad-projects/claude-micro/hardware/JLC.3dshapes/SOT-23-5_L2.9-W1.6-H1.1-LS2.8-P0.95.wrl"
+		(model "/Users/barakaeli/kicad-projects/agentdeck/hardware/JLC.3dshapes/SOT-23-5_L2.9-W1.6-H1.1-LS2.8-P0.95.wrl"
 			(offset
 				(xyz 0 0 0)
@@
 		)
 		(embedded_fonts no)
-		(model "/Users/barakaeli/kicad-projects/claude-micro/hardware/JLC.3dshapes/LED-SMD_4P-L3.2-W2.8-LS5.9_SK6812MINI-E.wrl"
+		(model "/Users/barakaeli/kicad-projects/agentdeck/hardware/JLC.3dshapes/LED-SMD_4P-L3.2-W2.8-LS5.9_SK6812MINI-E.wrl"
 			(offset
 				(xyz 0 0 0)
@@
 		)
 		(embedded_fonts no)
-		(model "/Users/barakaeli/kicad-projects/claude-micro/hardware/JLC.3dshapes/LED-SMD_4P-L3.2-W2.8-LS5.9_SK6812MINI-E.wrl"
+		(model "/Users/barakaeli/kicad-projects/agentdeck/hardware/JLC.3dshapes/LED-SMD_4P-L3.2-W2.8-LS5.9_SK6812MINI-E.wrl"
 			(offset
 				(xyz 0 0 0)
@@
 		)
 		(embedded_fonts no)
-		(model "/Users/barakaeli/kicad-projects/claude-micro/hardware/JLC.3dshapes/LED-SMD_4P-L3.2-W2.8-LS5.9_SK6812MINI-E.wrl"
+		(model "/Users/barakaeli/kicad-projects/agentdeck/hardware/JLC.3dshapes/LED-SMD_4P-L3.2-W2.8-LS5.9_SK6812MINI-E.wrl"
 			(offset
 				(xyz 0 0 0)
@@
 		)
 		(embedded_fonts no)
-		(model "/Users/barakaeli/kicad-projects/claude-micro/hardware/JLC.3dshapes/LED-SMD_4P-L3.2-W2.8-LS5.9_SK6812MINI-E.wrl"
+		(model "/Users/barakaeli/kicad-projects/agentdeck/hardware/JLC.3dshapes/LED-SMD_4P-L3.2-W2.8-LS5.9_SK6812MINI-E.wrl"
 			(offset
 				(xyz 0 0 0)
@@
 		)
 		(embedded_fonts no)
-		(model "/Users/barakaeli/kicad-projects/claude-micro/hardware/JLC.3dshapes/LED-SMD_4P-L3.2-W2.8-LS5.9_SK6812MINI-E.wrl"
+		(model "/Users/barakaeli/kicad-projects/agentdeck/hardware/JLC.3dshapes/LED-SMD_4P-L3.2-W2.8-LS5.9_SK6812MINI-E.wrl"
 			(offset
 				(xyz 0 0 0)
@@
 		)
 		(embedded_fonts no)
-		(model "/Users/barakaeli/kicad-projects/claude-micro/hardware/JLC.3dshapes/LED-SMD_4P-L3.2-W2.8-LS5.9_SK6812MINI-E.wrl"
+		(model "/Users/barakaeli/kicad-projects/agentdeck/hardware/JLC.3dshapes/LED-SMD_4P-L3.2-W2.8-LS5.9_SK6812MINI-E.wrl"
 			(offset
 				(xyz 0 0 0)
@@
 		)
 		(embedded_fonts no)
-		(model "/Users/barakaeli/kicad-projects/claude-micro/hardware/JLC.3dshapes/LED-SMD_4P-L3.2-W2.8-LS5.9_SK6812MINI-E.wrl"
+		(model "/Users/barakaeli/kicad-projects/agentdeck/hardware/JLC.3dshapes/LED-SMD_4P-L3.2-W2.8-LS5.9_SK6812MINI-E.wrl"
 			(offset
 				(xyz 0 0 0)
@@
 		)
 		(embedded_fonts no)
-		(model "/Users/barakaeli/kicad-projects/claude-micro/hardware/JLC.3dshapes/LED-SMD_4P-L3.2-W2.8-LS5.9_SK6812MINI-E.wrl"
+		(model "/Users/barakaeli/kicad-projects/agentdeck/hardware/JLC.3dshapes/LED-SMD_4P-L3.2-W2.8-LS5.9_SK6812MINI-E.wrl"
 			(offset
 				(xyz 0 0 0)
@@
 		)
 		(embedded_fonts no)
-		(model "/Users/barakaeli/kicad-projects/claude-micro/hardware/JLC.3dshapes/LED-SMD_4P-L3.2-W2.8-LS5.9_SK6812MINI-E.wrl"
+		(model "/Users/barakaeli/kicad-projects/agentdeck/hardware/JLC.3dshapes/LED-SMD_4P-L3.2-W2.8-LS5.9_SK6812MINI-E.wrl"
 			(offset
 				(xyz 0 0 0)
@@
 		)
 		(embedded_fonts no)
-		(model "/Users/barakaeli/kicad-projects/claude-micro/hardware/JLC.3dshapes/LED-SMD_4P-L3.2-W2.8-LS5.9_SK6812MINI-E.wrl"
+		(model "/Users/barakaeli/kicad-projects/agentdeck/hardware/JLC.3dshapes/LED-SMD_4P-L3.2-W2.8-LS5.9_SK6812MINI-E.wrl"
 			(offset
 				(xyz 0 0 0)
@@
 		)
 		(embedded_fonts no)
-		(model "/Users/barakaeli/kicad-projects/claude-micro/hardware/JLC.3dshapes/LED-SMD_4P-L3.2-W2.8-LS5.9_SK6812MINI-E.wrl"
+		(model "/Users/barakaeli/kicad-projects/agentdeck/hardware/JLC.3dshapes/LED-SMD_4P-L3.2-W2.8-LS5.9_SK6812MINI-E.wrl"
 			(offset
 				(xyz 0 0 0)
@@
 		)
 		(embedded_fonts no)
-		(model "/Users/barakaeli/kicad-projects/claude-micro/hardware/JLC.3dshapes/LED-SMD_4P-L3.2-W2.8-LS5.9_SK6812MINI-E.wrl"
+		(model "/Users/barakaeli/kicad-projects/agentdeck/hardware/JLC.3dshapes/LED-SMD_4P-L3.2-W2.8-LS5.9_SK6812MINI-E.wrl"
 			(offset
 				(xyz 0 0 0)
@@
 		)
 		(embedded_fonts no)
-		(model "/Users/barakaeli/kicad-projects/claude-micro/hardware/JLC.3dshapes/LED-SMD_4P-L3.2-W2.8-LS5.9_SK6812MINI-E.wrl"
+		(model "/Users/barakaeli/kicad-projects/agentdeck/hardware/JLC.3dshapes/LED-SMD_4P-L3.2-W2.8-LS5.9_SK6812MINI-E.wrl"
 			(offset
 				(xyz 0 0 0)
@@
 		)
 		(embedded_fonts no)
-		(model "/Users/barakaeli/kicad-projects/claude-micro/hardware/JLC.3dshapes/LED-SMD_4P-L3.2-W2.8-LS5.9_SK6812MINI-E.wrl"
+		(model "/Users/barakaeli/kicad-projects/agentdeck/hardware/JLC.3dshapes/LED-SMD_4P-L3.2-W2.8-LS5.9_SK6812MINI-E.wrl"
 			(offset
 				(xyz 0 0 0)
@@
 		)
 	)
-	(gr_text "ClaudeMicro V4 - princetekki.com"
+	(gr_text "AgentDeck V4 - princetekki.com"
 		(at 24 106.3 0)
 		(layer "F.SilkS")
@@
 		)
 	)
-	(gr_text "ClaudeMicroV4  ESP32-S3-WROOM-1"
+	(gr_text "AgentDeckV4  ESP32-S3-WROOM-1"
 		(at 119 7 0)
 		(layer "B.SilkS")
