File: v4/hardware/AgentDeckV4.kicad_sch (KiCad schematic)
At the start: 136 parts, among them J1 TYPE-C-31-M-12, J2 JST-PH-2 LiPo, J3 ProgPads 3V3/TX/GND/RX, Q1 AO3401A, SW1 ChocV1, SW10 ChocV1, SW11 ChocV1, SW12 ChocV1, SW13 ChocV1, SW14 ChocV1, SW15 ChocV1, SW16 ChocV1, SW17 ChocV1, SW18 ChocV1, SW19 ChocV1, SW2 ChocV1, SW20 ChocV1, SW21 ChocV1, SW22 ChocV1, SW23 ChocV1, SW24 ChocV1, SW25 MSK12C02, SW26 SW_PUSH, SW27 SW_PUSH, SW3 ChocV1, SW4 ChocV1, SW5 ChocV1, SW6 ChocV1, SW7 ChocV1, SW8 ChocV1, SW9 ChocV1, U1 ESP32-S3-WROOM-1-N8R2, U2 SN74AHCT1G125, U3 USBLC6-2SC6, U4 TP4056, U5 ME6211C33

Commit message: rename to agentdeck 1.0.0
The product is renamed from ClaudeMicro to AgentDeck for 1.0.0. "Claude" is
Anthropic's trademark and this ships as OSHWA-marked open hardware with the
name on the silk; "Micro" also stopped describing a 150x110 mm V4 deck. Note
AgentDeck collides with an existing project (github.com/puritysb/AgentDeck) -
chosen anyway.

Renamed across board, schematic, netlist, libraries, firmware, host bridge and
docs. Silk reads AGENTDECK and AgentDeck v1.0.0. Generated gerbers under
fab/gerbers are left alone: they are the artifact of the released v0.1.0 and
should be regenerated rather than string-edited.

Also in this commit, all verified 0 errors / 0 unconnected:

- silkscreen pass (tools/silk_pass.py, silk_finish.py, fix_silk_font.py):
  silk_over_copper 79 -> 0, silk_overlap 7 -> 0, text_height 4 -> 0. Silk is
  Red Hat Mono bold; bold and 1.3 mm on the three longest strings are not
  cosmetic - KiCad flags Red Hat Mono Regular at 1.0 mm as insufficient stroke
  weight, the outline-font tradeoff a stroke font avoids. Re-running the pass
  is a no-op, so it is safe after any placement change.

- placement pass (tools/placement_pass.py): three fiducials placed
  asymmetrically >=5 mm from the edges, and C10 moved +0.75/-2.25 mm. C9 and
  C10 were not merely close, their bodies overlapped - two 0603 caps in the
  same space, invisible to DRC because both are +3V3/GND so no clearance rule
  applies. Only C10 moved; the outline and every part the case mates with are
  untouched.

- fab/AgentDeck-BOM-v1.0.0.csv. Records that C22967 is 27k, not the 27R the
  old BOM claimed for the USB series resistors - at 27k USB would not
  enumerate. Correct part is C25190. Also records what LCSC cannot supply:
  the Kailh hot-swap socket (C5333465 discontinued) and the SKQUCAA010
  joystick, plus switches and keycaps which were never LCSC lines.

- docs/img: top and bottom board renders.
Parts:
- removed J1: TYPE-C-31-M-12, JLC_V1:USB-C_SMD-TYPE-C-31-M-12_1, symbol V3:TYPE-C-31-M-12
- removed J3: ProgPads 3V3/TX/GND/RX, ClaudeMicro:ProgPads_1x4, symbol ClaudeMicro_Custom:ProgPads_1x4
- removed OLED1: HS96L03W2C03, V3:OLED_HS96L03, symbol V3:OLED_HS96L03
- removed Q1: AO3401A, Package_TO_SOT_SMD:SOT-23, symbol V3:AO3401A
- removed R4, R5: 10k, Resistor_SMD:R_0603_1608Metric, symbol Device:R
- removed SW1, SW10, SW11, SW12, SW13, SW14, SW15, SW16, SW17, SW18, SW19, SW2, SW20, SW21, SW22, SW23, SW24, SW3, SW4, SW5, SW6, SW7, SW8, SW9: ChocV1, V3:ChocV1_Direct, symbol V3:ChocV1
- removed SW25: MSK12C02, V3:MSK12C02, symbol V3:MSK12C02
- removed SW26, SW27: SW_PUSH, JLC_V1:SW-SMD_4P-L5.1-W5.1-P3.70-LS6.5-TL_H1.5, symbol V3:TS-1187A-B-A-B
- removed TP1: TouchPad, ClaudeMicro:TouchPad_D12, symbol ClaudeMicro_Custom:TouchPad
- removed U1: ESP32-S3-WROOM-1-N8R2, V3:WIRELM-SMD_ESP32-S3-WROOM-1, symbol V3:ESP32-S3-WROOM-1
- removed U3: USBLC6-2SC6, JLC_V1:SOT-23-6_L2.9-W1.6-P0.95-LS2.8-BL, symbol V3:USBLC6-2SC6
- removed U4: TP4056, V3:ESOP-8_TP4056, symbol V3:TP4056
- removed U5: ME6211C33, JLC_V1:SOT-23-5_L3.0-W1.7-P0.95-LS2.8-BR, symbol V3:ME6211C33M5G-N
- added C36, C38: 100nF, Capacitor_SMD:C_0603_1608Metric, symbol Device:C
- added C37: 22uF, Capacitor_SMD:C_0805_2012Metric, symbol Device:C
- added ENC2: EC11, JLC_V1:SW-TH_EC11E1820402, symbol JLC_V1:EC11E1834403
- added J1: TYPE-C-31-M-12, JLC_V1:USB-C_SMD-TYPE-C-31-M-12_1, symbol V4:TYPE-C-31-M-12
- added J3: ProgPads 3V3/TX/GND/RX, AgentDeck:ProgPads_1x4, symbol AgentDeck_Custom:ProgPads_1x4
- added J4: JST-PH-2 Speaker, Connector_JST:JST_PH_S2B-PH-SM4-TB_1x02-1MP_P2.00mm_Horizontal, symbol Connector_Generic:Conn_01x02
- added LCD1: LCD_169_Touch, V4:LCD_1x12_2p54_Module, symbol V4:LCD_169_Touch
- added MK1: MEMS_Mic_I2S, V4:MEMS_Mic_I2S_3p5x2p65, symbol V4:MEMS_Mic_I2S
- added Q1: AO3401A, Package_TO_SOT_SMD:SOT-23, symbol V4:AO3401A
- added R14: 100R, Resistor_SMD:R_0603_1608Metric, symbol Device:R
- added SW1, SW10, SW11, SW12, SW13, SW14, SW15, SW16, SW17, SW18, SW19, SW2, SW20, SW21, SW22, SW23, SW24, SW3, SW4, SW5, SW6, SW7, SW8, SW9: ChocV1, V3:ChocV1_Direct, symbol V4:ChocV1
- added SW25: MSK12C02, V3:MSK12C02, symbol V4:MSK12C02
- added SW26, SW27: SW_PUSH, JLC_V1:SW-SMD_4P-L5.1-W5.1-P3.70-LS6.5-TL_H1.5, symbol V4:TS-1187A-B-A-B
- added TP1: TouchPad, AgentDeck:TouchPad_D12, symbol AgentDeck_Custom:TouchPad
- added U1: ESP32-S3-WROOM-1-N8R2, V3:WIRELM-SMD_ESP32-S3-WROOM-1, symbol V4:ESP32-S3-WROOM-1
- added U3: USBLC6-2SC6, JLC_V1:SOT-23-6_L2.9-W1.6-P0.95-LS2.8-BL, symbol V4:USBLC6-2SC6
- added U4: TP4056, V3:ESOP-8_TP4056, symbol V4:TP4056
- added U5: ME6211C33, JLC_V1:SOT-23-5_L3.0-W1.7-P0.95-LS2.8-BR, symbol V4:ME6211C33M5G-N
- added U6: NS4168, V4:ESOP-8_NS4168, symbol V4:NS4168
Connections:
- net +3V3: now also C38.1, J3.1 (SWCLK), LCD1.1 (VCC), MK1.1 (VDD), R14.1, U1.2 (3V3), U5.5 (VOUT)
- net BAT+: now also Q1.3 (D), U4.5 (BAT)
- net CC1: now also J1.A5 (CC1)
- net CC2: now also J1.B5 (CC2)
- net COL0: now also SW1.1, SW13.1, SW19.1, SW7.1, U1.18 (IO10)
- net COL1: now also SW14.1, SW2.1, SW20.1, SW8.1, U1.19 (IO11)
- net COL2: now also SW15.1, SW21.1, SW3.1, SW9.1, U1.20 (IO12)
- net COL3: now also SW10.1, SW16.1, SW22.1, SW4.1, U1.21 (IO13)
- net COL4: now also SW11.1, SW17.1, SW23.1, SW5.1, U1.22 (IO14)
- net COL5: now also SW12.1, SW18.1, SW24.1, SW6.1, U1.8 (IO15)
- net EN: now also LCD1.12 (TP_RST), LCD1.7 (RST), SW27.1 (A), SW27.3 (C), U1.3 (EN)
- net GND: now also C36.2, C37.2, C38.2, ENC2.C, ENC2.E, ENC2.F, ENC2.G, J1.1 (EH), J1.2 (EH), J1.3 (EH), J1.4 (EH), J1.A1B12 (GND), J1.B1A12 (GND), J3.3 (GND), LCD1.2 (GND), LCD1.5 (CS), MK1.2 (GND), MK1.6 (LR), SW26.2 (B), SW26.4 (D), SW27.2 (B), SW27.4 (D), U1.1 (GND), U1.40 (GND), U1.41 (GND), U3.2, U4.1 (TEMP), U4.3 (GND), U5.2 (VSS), U6.7 (GND)
- net IO0: now also SW26.1 (A), SW26.3 (C), U1.27 (IO0)
- net KD1: now also SW1.2
- net KD10: now also SW10.2
- net KD11: now also SW11.2
- net KD12: now also SW12.2
- net KD13: now also SW13.2
- net KD14: now also SW14.2
- net KD15: now also SW15.2
- net KD16: now also SW16.2
- net KD17: now also SW17.2
- net KD18: now also SW18.2
- net KD19: now also SW19.2
- net KD2: now also SW2.2
- net KD20: now also SW20.2
- net KD21: now also SW21.2
- net KD22: now also SW22.2
- net KD23: now also SW23.2
- net KD24: now also SW24.2
- net KD3: now also SW3.2
- net KD4: now also SW4.2
- net KD5: now also SW5.2
- net KD6: now also SW6.2
- net KD7: now also SW7.2
- net KD8: now also SW8.2
- net KD9: now also SW9.2
- net LED_DATA: now also U1.23 (IO21)
- net PROG: now also U4.2 (PROG)
- net ROW0: now also U1.4 (IO4)
- net ROW1: now also U1.5 (IO5)
- net ROW2: now also U1.6 (IO6)
- net ROW3: now also U1.7 (IO7)
- net RXD: now also J3.4 (RUN), U1.36 (RXD0)
- net SCL: now also LCD1.10 (TP_SCL), U1.17 (IO9)
- net SDA: now also LCD1.9 (TP_SDA), U1.12 (IO8)
- net TOUCH: now also TP1.1 (PAD), U1.39 (IO1)
- net TXD: now also J3.2 (SWDIO), U1.37 (TXD0)
- net USB_DM: now also J1.A7 (DN1), J1.B7 (DN2), U1.13 (IO19), U3.1, U3.6
- net USB_DP: now also J1.A6 (DP1), J1.B6 (DP2), U1.14 (IO20), U3.3, U3.4
- net VBAT_SNS: now also U1.38 (IO2)
- net VBUS: now also J1.A4B9 (VBUS), J1.B4A9 (VBUS), Q1.1 (G), U3.5, U4.4 (VCC), U4.8 (CE)
- net VSYS: now also Q1.2 (S), SW25.2 (COM)
- net VSYS_SW: now also C36.1, C37.1, SW25.1 (A), U5.1 (VIN), U5.3 (CE), U6.1 (CTRL), U6.6 (VDD)
- net ENC_A renamed ENC1_A
- net ENC1_A: now also U1.33 (IO40)
- net ENC_B renamed ENC1_B
- net ENC1_B: now also U1.34 (IO41)
- net ENC_SW renamed ENC1_SW
- net ENC1_SW: now also U1.35 (IO42)
- new net AMP_OUTN: J4.2 (Pin_2), U6.5 (VoN)
- new net AMP_OUTP: J4.1 (Pin_1), U6.8 (VoP)
- new net ENC2_A: ENC2.A, U1.28 (IO35)
- new net ENC2_B: ENC2.B, U1.29 (IO36)
- new net ENC2_SW: ENC2.D, U1.30 (IO37)
- new net I2S_BCLK: MK1.3 (BCLK), U1.31 (IO38), U6.3 (BCLK)
- new net I2S_DIN: MK1.5 (SD), U1.25 (IO48)
- new net I2S_DOUT: U1.24 (IO47), U6.4 (SDATA)
- new net I2S_WS: MK1.4 (WS), U1.32 (IO39), U6.2 (LRCLK)
- new net LCD_BL: LCD1.8 (BL), R14.2
- new net LCD_DC: LCD1.6 (DC), U1.11 (IO18)
- new net LCD_MOSI: LCD1.3 (DIN), U1.10 (IO17)
- new net LCD_SCK: LCD1.4 (CLK), U1.9 (IO16)
- no-connect marks 16 -> 11
Other:
- note added: "AUDIO (U6 NS4168 I2S 2.5W amp @VSYS_SW -> J4 speaker + MK1 I2S MEMS mic)"
- note added: "PERIPHERALS (1.69in touch LCD SPI/I2C + touch pad + 2x EC11)"
- note removed: "PERIPHERALS (OLED I2C + touch pad + EC11)"
- title: ClaudeMicroV3 -> AgentDeckV4
