File: v2/hardware/AgentDeckV2.kicad_sch (KiCad schematic)
At the start: 126 parts, among them J1 TYPE-C-31-M-12, J2 JST-PH-2 LiPo, J3 ProgPads 3V3/TX/GND/RX, Q1 AO3401A, Q2 AO3400A, SW1 ChocV1, SW10 ChocV1, SW11 ChocV1, SW12 ChocV1, SW13 ChocV1, SW14 ChocV1, SW15 ChocV1, SW16 ChocV1, SW17 ChocV1, SW18 ChocV1, SW19 ChocV1, SW2 ChocV1, SW20 ChocV1, SW25 MSK12C02, SW26 SW_PUSH, SW27 SW_PUSH, SW3 ChocV1, SW4 ChocV1, SW5 ChocV1, SW6 ChocV1, SW7 ChocV1, SW8 ChocV1, SW9 ChocV1, U1 ESP32-S3-WROOM-1-N8R2, U2 SN74AHCT1G125, U3 USBLC6-2SC6, U4 TP4056, U5 ME6211C33

Commit message: place v2 board
Parts:
- Q2: footprint JLC:SOT-23-3P_L2.9-W1.3-H1.0-LS2.4-P0.95 -> JLC:SOT-23-3_L2.9-W1.3-P1.90-LS2.4-BR
Changed lines of the file:
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@@
 			)
 		)
-		(property "Footprint" "JLC:SOT-23-3P_L2.9-W1.3-H1.0-LS2.4-P0.95"
+		(property "Footprint" "JLC:SOT-23-3_L2.9-W1.3-P1.90-LS2.4-BR"
 			(at 375.0 240.0 0)
 			(effects

Commit message: remove v2 lcd battery
Parts:
- removed C10, C8: 100nF, Capacitor_SMD:C_0603_1608Metric, symbol Device:C
- removed C11: 10uF, Capacitor_SMD:C_0805_2012Metric, symbol Device:C
- removed D26: SS34, Diode_SMD:D_SMA, symbol Device:D
- removed J2: JST-PH-2 LiPo, JLC:CONN-SMD_P2.00_S2B-PH-SM4-TB-LF-SN, symbol Connector_Generic:Conn_01x02
- removed LCD1: N114-2413THBIG01-H13, JLC:LCD-SMD_1.14IPS-LCD, symbol V2:N114-2413THBIG01-H13
- removed Q1: AO3401A, Package_TO_SOT_SMD:SOT-23, symbol V2:AO3401A
- removed Q2: AO3400A, JLC:SOT-23-3_L2.9-W1.3-P1.90-LS2.4-BR, symbol V2:AO3400A
- removed R12: 22R, Resistor_SMD:R_0603_1608Metric, symbol Device:R
- removed R13, R4, R5: 10k, Resistor_SMD:R_0603_1608Metric, symbol Device:R
- removed R3: 1.2k, Resistor_SMD:R_0603_1608Metric, symbol Device:R
- removed R6, R7: 100k, Resistor_SMD:R_0603_1608Metric, symbol Device:R
- removed R8: 47k, Resistor_SMD:R_0603_1608Metric, symbol Device:R
- removed SW25: MSK12C02, V3:MSK12C02, symbol V2:MSK12C02
- removed U4: TP4056, JLC:ESOP-8_L4.9-W3.9-P1.27-LS6.0-BL-EP, symbol V2:TP4056
Connections:
- net VSYS_SW is gone; now on net VBUS: C12.1, C13.1, C14.1, C15.1, C16.1, C17.1, C18.1, C19.1, C20.1, C21.1, C22.1, C23.1, C24.1, C25.1, C26.1, C27.1, C28.1, C29.1, C30.1, C31.1, C6.1, C9.1, LED1.3 (VDD), LED10.3 (VDD), LED11.3 (VDD), LED12.3 (VDD), LED13.3 (VDD), LED14.3 (VDD), LED15.3 (VDD), LED16.3 (VDD), LED17.3 (VDD), LED18.3 (VDD), LED19.3 (VDD), LED2.3 (VDD), LED20.3 (VDD), LED3.3 (VDD), LED4.3 (VDD), LED5.3 (VDD), LED6.3 (VDD), LED7.3 (VDD), LED8.3 (VDD), LED9.3 (VDD), U2.5 (VCC), U5.1 (VIN), U5.3 (CE)
- net CHRG_SNS: no longer names the net of U1.24 (IO47)
- net LCD_BL: no longer names the net of U1.39 (IO1)
- net LCD_CS: no longer names the net of U1.10 (IO17)
- net LCD_DC: no longer names the net of U1.9 (IO16)
- net LCD_MOSI: no longer names the net of U1.12 (IO8)
- net LCD_RST: no longer names the net of U1.11 (IO18)
- net LCD_SCK: no longer names the net of U1.17 (IO9)
- net STDBY_SNS: no longer names the net of U1.25 (IO48)
- net VBAT_SNS: no longer names the net of U1.38 (IO2)
- no-connect marks 16 -> 21
Other:
- note added: "PERIPHERALS (EC11 encoder)"
- note added: "POWER (USB-C + ESD + ME6211 3V3, VBUS LED rail)"
- note added: "RGB LEDs (U2 AHCT125 @VBUS + 330R head + 20x SK6812MINI-E, 100nF each)"
- note removed: "PERIPHERALS (1.14in ST7789V SPI LCD + EC11)"
- note removed: "POWER (USB-C + TP4056 charge + AO3401A load-share + MSK12C02 switch + ME6211 3V3)"
- note removed: "RGB LEDs (U2 AHCT125 @VSYS_SW + 330R head + 20x SK6812MINI-E, 100nF each)"
