File: v2/hardware/AgentDeckV2.kicad_sch (KiCad schematic)
At the start: 120 parts, among them J1 TYPE-C-31-M-12, J2 JST-PH-2 LiPo, J3 ProgPads 3V3/TX/GND/RX, Q1 AO3401A, SW1 ChocV1, SW10 ChocV1, SW11 ChocV1, SW12 ChocV1, SW13 ChocV1, SW14 ChocV1, SW15 ChocV1, SW16 ChocV1, SW17 ChocV1, SW18 ChocV1, SW19 ChocV1, SW2 ChocV1, SW20 ChocV1, SW25 MSK12C02, SW26 SW_PUSH, SW27 SW_PUSH, SW3 ChocV1, SW4 ChocV1, SW5 ChocV1, SW6 ChocV1, SW7 ChocV1, SW8 ChocV1, SW9 ChocV1, U1 ESP32-S3-WROOM-1-N8R2, U2 SN74AHCT1G125, U3 USBLC6-2SC6, U4 TP4056, U5 ME6211C33

Commit message: source v2 from jlcpcb
Every LCSC code re-checked against the JLCPCB assembly library; LCSC
field on all symbols; JLCPCB BOM/CPL/consigned list in v2/fab. LDO ->
RT9080-33GJ5 (ME6211 had 17 in stock), joystick -> SKRHABE010 SMD with
the JLC library footprint. STEP models pulled per LCSC code.

Claude-Session: https://claude.ai/code/session_01GWeFSftAaDQLi7MhELLoa4
Parts:
- removed JS1: SKQUCAA010, AgentDeck:SKQUCAA010, symbol AgentDeck_Custom:SKQUCAA010
- added JS1: SKRHABE010, V2:SW-SMD_SKRHABE010, symbol JLC_V1:SKRHABE010
- C1, C10, C12, C13, C14, C15, C16, C17, C18, C19, C2, C20, C21, C22, C23, C24, C25, C26, C27, C28, C29, C3, C30, C31, C5, C8, C9: LCSC (none) -> C14663
- C11, C4: LCSC (none) -> C15850
- C6, C7: LCSC (none) -> C28323
- D1, D10, D11, D12, D13, D14, D15, D16, D17, D18, D19, D2, D20, D3, D4, D5, D6, D7, D8, D9: LCSC (none) -> C81598
- D25: LCSC (none) -> C8678
- ENC1: LCSC (none) -> C361165
- J1: LCSC (none) -> C165948
- J2: LCSC (none) -> C295747
- LED1, LED10, LED11, LED12, LED13, LED14, LED15, LED16, LED17, LED18, LED19, LED2, LED20, LED3, LED4, LED5, LED6, LED7, LED8, LED9: LCSC (none) -> C5149201
- Q1: LCSC (none) -> C15127
- R1, R2: LCSC (none) -> C23186
- R10, R4, R5, R9: LCSC (none) -> C25804
- R11: LCSC (none) -> C23138
- R12, R13: LCSC (none) -> C23162
- R3: LCSC (none) -> C22940
- R6, R7: LCSC (none) -> C25803
- R8: LCSC (none) -> C25819
- SW1, SW10, SW11, SW12, SW13, SW14, SW15, SW16, SW17, SW18, SW19, SW2, SW20, SW3, SW4, SW5, SW6, SW7, SW8, SW9: LCSC (none) -> C400229
- SW25: LCSC (none) -> C431540
- SW26, SW27: LCSC (none) -> C318884
- U1: LCSC (none) -> C2913204
- U2: LCSC (none) -> C7484
- U3: LCSC (none) -> C7519
- U4: LCSC (none) -> C16581
- U5: value ME6211C33 -> RT9080-33GJ5; LCSC (none) -> C841192
Connections:
- net GND: now also JS1.5 (COM)
- net JOY_CTR: now also JS1.2 (CEN)
- net JOY_DOWN: now also JS1.3 (C)
- net JOY_LEFT: now also JS1.6 (B)
- net JOY_RIGHT: now also JS1.4 (D)
- net JOY_UP: now also JS1.1 (A)
- no-connect marks 13 -> 15

Commit message: oled from jlcpcb library
C5248080 module with JLC footprint and STEP replaces the stand-in and the
generated model; OLED joins the JLCPCB BOM.

Claude-Session: https://claude.ai/code/session_01GWeFSftAaDQLi7MhELLoa4
Parts:
- OLED1: footprint V2:OLED_HS96L03 -> V2:OLED-TH_HS96L03_C5248080; LCSC (none) -> C5248080
Changed lines of the file:
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@@
 			)
 		)
-		(property "Footprint" "V2:OLED_HS96L03"
+		(property "Footprint" "V2:OLED-TH_HS96L03_C5248080"
 			(at 330.0 180.0 0)
 			(effects
@@
 			(hide yes)
 		)
-		(property "LCSC" ""
+		(property "LCSC" "C5248080"
 			(at 330.0 180.0 0)
 			(effects
