File: v2/hardware/AgentDeckV2.kicad_pcb (KiCad board)
At the start: 2 copper layers, 112 x 112 mm, 130 parts, among them J1 USB-C_SMD-TYPE-C-31-M-12_1, J2 CONN-SMD_P2.00_S2B-PH-SM4-TB-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, J3 SWD, Q1 SOT-23, Q2 SOT-23-3_L2.9-W1.3-P1.90-LS2.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, SW1 CONN-SMD_HOTPLUGPAKAGE__C9900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, SW10 CONN-SMD_HOTPLUGPAKAGE__C9900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, SW11 CONN-SMD_HOTPLUGPAKAGE__C9900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, SW12 CONN-SMD_HOTPLUGPAKAGE__C9900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, SW13 CONN-SMD_HOTPLUGPAKAGE__C9900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, SW14 CONN-SMD_HOTPLUGPAKAGE__C9900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, SW15 CONN-SMD_HOTPLUGPAKAGE__C9900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, SW16 CONN-SMD_HOTPLUGPAKAGE__C9900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, SW17 CONN-SMD_HOTPLUGPAKAGE__C9900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, SW18 CONN-SMD_HOTPLUGPAKAGE__C9900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, SW19 CONN-SMD_HOTPLUGPAKAGE__C9900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, SW2 CONN-SMD_HOTPLUGPAKAGE__C9900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, SW20 CONN-SMD_HOTPLUGPAKAGE__C9900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, SW25 MSK12C02, SW26 SW-SMD_4P-L5.1-W5.1-P3.70-LS6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, SW27 SW-SMD_4P-L5.1-W5.1-P3.70-LS6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, SW3 CONN-SMD_HOTPLUGPAKAGE__C9900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, SW4 CONN-SMD_HOTPLUGPAKAGE__C9900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, SW5 CONN-SMD_HOTPLUGPAKAGE__C9900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, SW6 CONN-SMD_HOTPLUGPAKAGE__C9900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, SW7 CONN-SMD_HOTPLUGPAKAGE__C9900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, SW8 CONN-SMD_HOTPLUGPAKAGE__C9900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, SW9 CONN-SMD_HOTPLUGPAKAGE__C9900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, U1 WIRELM-SMD_ESP32-S3-WROOM-1, U2 SOT-23-5_L3.0-W1.7-P0.95-LS2.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, U3 SOT-23-6_L2.9-W1.6-P0.95-LS2.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, U4 ESOP-8_L4.9-W3.9-P1.27-LS6.0-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, U5 SOT-23-5_L3.0-W1.7-P0.95-LS2.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

Commit message: route v2 board clean
Parts:
- moved Q1 7.07 mm to (106.5, 13.0), turned to 90 degrees
- moved R6 6.36 mm to (99.5, 19.0)
- moved ENC1 2.00 mm to (39.0, 13.0)
Routing:
- net +3V3: track 0.00 -> 208.9 mm, vias 0 -> 7
- net COL2: track 0.00 -> 171.9 mm, vias 0 -> 7
- net ROW3: track 0.00 -> 167.5 mm, vias 0 -> 6
- net COL0: track 0.00 -> 166.9 mm, vias 0 -> 6
- net COL1: track 0.00 -> 162.3 mm, vias 0 -> 7
- net COL4: track 0.00 -> 161.4 mm, vias 0 -> 6
- net COL3: track 0.00 -> 153.5 mm, vias 0 -> 7
- net ROW2: track 0.00 -> 151.9 mm, vias 0 -> 6
- net ROW1: track 0.00 -> 141.5 mm, vias 0 -> 6
- net ROW0: track 0.00 -> 116.2 mm, vias 0 -> 6
- net VBAT_SNS: track 0.00 -> 106.9 mm, vias 0 -> 3
- net USB_DP: track 0.00 -> 97.6 mm, vias 0 -> 5
- net USB_DM: track 0.00 -> 84.9 mm, vias 0 -> 3
- net ROW4: track 0.00 -> 84.1 mm, vias 0 -> 1
- net VBUS: track 6.86 -> 86.8 mm, vias 2 -> 6
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- added copper zone on B.Cu, net GND
- added copper zone on F.Cu, net GND
- added copper zone on In1.Cu, net GND
- added copper zone on In2.Cu, net GND
- added copper zone on B.Cu, net VSYS_SW
Other:
- copper layers 2 -> 4

Commit message: remove v2 lcd battery
Parts:
- removed C10, C8: C_0603_1608Metric, C_0603_1608Metric
- removed C11: C_0805_2012Metric, C_0805_2012Metric
- removed D26: D_SMA, D_SMA
- removed J2: CONN-SMD_P2.00_S2B-PH-SM4-TB-LF-SN, CONN-SMD_P2.00_S2B-PH-SM4-TB-LF-SN
- removed LCD1: LCD-SMD_1.14IPS-LCD, LCD-SMD_1.14IPS-LCD
- removed Q1: SOT-23, SOT-23
- removed Q2: SOT-23-3_L2.9-W1.3-P1.90-LS2.4-BR, SOT-23-3_L2.9-W1.3-P1.90-LS2.4-BR
- removed R12, R13, R3, R4, R5, R6, R7, R8: R_0603_1608Metric, R_0603_1608Metric
- removed SW25: MSK12C02, MSK12C02
- removed U4: ESOP-8_L4.9-W3.9-P1.27-LS6.0-BL-EP, ESOP-8_L4.9-W3.9-P1.27-LS6.0-BL-EP
- moved C6 14.5 mm to (94.0, 15.0)
- moved C7 14.5 mm to (103.5, 15.0)
- moved U5 14.5 mm to (99.0, 10.0)
Connections:
- C12 pad 1: VSYS_SW -> VBUS
- C13 pad 1: VSYS_SW -> VBUS
- C14 pad 1: VSYS_SW -> VBUS
- C15 pad 1: VSYS_SW -> VBUS
- C16 pad 1: VSYS_SW -> VBUS
- C17 pad 1: VSYS_SW -> VBUS
- C18 pad 1: VSYS_SW -> VBUS
- C19 pad 1: VSYS_SW -> VBUS
- C20 pad 1: VSYS_SW -> VBUS
- C21 pad 1: VSYS_SW -> VBUS
- C22 pad 1: VSYS_SW -> VBUS
- C23 pad 1: VSYS_SW -> VBUS
- C24 pad 1: VSYS_SW -> VBUS
- C25 pad 1: VSYS_SW -> VBUS
- C26 pad 1: VSYS_SW -> VBUS
- C27 pad 1: VSYS_SW -> VBUS
- C28 pad 1: VSYS_SW -> VBUS
- C29 pad 1: VSYS_SW -> VBUS
- C30 pad 1: VSYS_SW -> VBUS
- C31 pad 1: VSYS_SW -> VBUS
- C6 pad 1: VSYS_SW -> VBUS
- C9 pad 1: VSYS_SW -> VBUS
- LED1 pad 3: VSYS_SW -> VBUS
- LED10 pad 3: VSYS_SW -> VBUS
- LED11 pad 3: VSYS_SW -> VBUS
- LED12 pad 3: VSYS_SW -> VBUS
- LED13 pad 3: VSYS_SW -> VBUS
- LED14 pad 3: VSYS_SW -> VBUS
- LED15 pad 3: VSYS_SW -> VBUS
- LED16 pad 3: VSYS_SW -> VBUS
- LED17 pad 3: VSYS_SW -> VBUS
- LED18 pad 3: VSYS_SW -> VBUS
- LED19 pad 3: VSYS_SW -> VBUS
- LED2 pad 3: VSYS_SW -> VBUS
- LED20 pad 3: VSYS_SW -> VBUS
- LED3 pad 3: VSYS_SW -> VBUS
- LED4 pad 3: VSYS_SW -> VBUS
- LED5 pad 3: VSYS_SW -> VBUS
- LED6 pad 3: VSYS_SW -> VBUS
- LED7 pad 3: VSYS_SW -> VBUS
- LED8 pad 3: VSYS_SW -> VBUS
- LED9 pad 3: VSYS_SW -> VBUS
- U1 pad 10: LCD_CS -> unconnected-(U1-IO17-Pad10)
- U1 pad 11: LCD_RST -> unconnected-(U1-IO18-Pad11)
- U1 pad 12: LCD_MOSI -> unconnected-(U1-IO8-Pad12)
- U1 pad 17: LCD_SCK -> unconnected-(U1-IO9-Pad17)
- U1 pad 24: CHRG_SNS -> unconnected-(U1-IO47-Pad24)
- U1 pad 25: STDBY_SNS -> unconnected-(U1-IO48-Pad25)
- U1 pad 38: VBAT_SNS -> unconnected-(U1-IO2-Pad38)
- U1 pad 39: LCD_BL -> unconnected-(U1-IO1-Pad39)
- U1 pad 9: LCD_DC -> unconnected-(U1-IO16-Pad9)
- U2 pad 5: VSYS_SW -> VBUS
- U5 pad 1: VSYS_SW -> VBUS
- U5 pad 3: VSYS_SW -> VBUS
Routing:
- net VBAT_SNS: track 106.9 -> 0.00 mm, vias 3 -> 0
- net CHRG_SNS: track 74.5 -> 0.00 mm, vias 2 -> 0
- net STDBY_SNS: track 72.4 -> 0.00 mm, vias 2 -> 0
- net LCD_CS: track 67.1 -> 0.00 mm, vias 3 -> 0
- net LCD_RST: track 59.7 -> 0.00 mm, vias 3 -> 0
- net LCD_DC: track 58.7 -> 0.00 mm, vias 3 -> 0
- net LCD_MOSI: track 58.4 -> 0.00 mm, vias 2 -> 0
- net LCD_SCK: track 57.0 -> 0.00 mm, vias 2 -> 0
- net LCD_BL: track 55.8 -> 0.00 mm, vias 2 -> 0
- net VSYS: track 52.3 -> 0.00 mm, vias 3 -> 0
- net BAT+: track 46.6 -> 0.00 mm, vias 4 -> 0
- net LCD_LEDA: track 41.0 -> 0.00 mm, vias 2 -> 0
- net VBUS: track 86.8 -> 58.7 mm, vias 6 -> 50
- net +3V3: track 208.9 -> 181.5 mm, vias 7 -> 4
- net LCD_LEDK: track 27.5 -> 0.00 mm, vias 2 -> 0
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- added copper zone on B.Cu, net VBUS
- removed copper zone on B.Cu, net VSYS_SW
Other:
- board text added: "LED=IO21 ENC A/B/SW=IO40/41/42"
- board text removed: "BAT"
- board text removed: "BATTERY 103450 2000mAh IN TRAY BELOW - KEEP FLAT"
- board text removed: "LCD GLASS"
- board text removed: "LCD MOSI/SCK/DC/CS/RST=IO8/9/16/17/18 BL=IO1"
- board text removed: "LED=IO21 ENC A/B/SW=IO40/41/42 VBAT=IO2"
- board text removed: "PWR"

Commit message: flip sockets add fab
Parts:
- SW1, SW10, SW11, SW12, SW13, SW14, SW15, SW16, SW17, SW18, SW19, SW2, SW20, SW3, SW4, SW5, SW6, SW7, SW8, SW9: moved to B.Cu
Routing:
- net VBUS: track 58.7 -> 93.5 mm
- net COL0: track 167.4 -> 160.3 mm
- net JS_RIGHT: track 22.6 -> 16.4 mm
- net USB_DP: track 89.0 -> 83.6 mm
- net KD18: track 12.2 -> 17.5 mm, vias 1 -> 2
- net KD13: track 11.8 -> 16.2 mm
- net COL3: track 155.3 -> 159.5 mm, vias 7 -> 6
- net KD8: track 13.7 -> 17.8 mm
- net COL1: track 161.1 -> 157.1 mm, vias 7 -> 6
- net LED_D2: track 13.9 -> 17.6 mm, vias 0 -> 2
- net LED_D3: track 13.9 -> 17.6 mm, vias 0 -> 2
- net KD3: track 12.9 -> 16.2 mm
- net COL4: track 155.7 -> 152.5 mm
- net LED_D17: track 20.2 -> 17.4 mm
- net LED_D18: track 13.9 -> 16.6 mm, vias 0 -> 2
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